Commit message: Rename to supermarketbot: supermarket world, customer detection, full project rebrand

File: supermarketbot/urdf/supermarketbot.xacro (robot description, xacro)
@@ -1,4 +1,4 @@
 <?xml version="1.0" ?>
-<robot xmlns:xacro="http://www.ros.org/wiki/xacro" name="amr_fe01">
+<robot xmlns:xacro="http://www.ros.org/wiki/xacro" name="supermarketbot">
   <!--some materials-->
   <xacro:property name="black" value="0.02 0.02 0.02 1.0" />
@@ -20,5 +20,5 @@
       <origin xyz="0 0 0" rpy="0 0 0" />
       <geometry>
-        <mesh filename="package://amr_fe01/meshes/chassis_l1.stl" scale="0.001 0.001 0.001" />
+        <mesh filename="package://supermarketbot/meshes/chassis_l1.stl" scale="0.001 0.001 0.001" />
       </geometry>
       <material name="1">
@@ -29,5 +29,5 @@
       <origin xyz="0 0 0" rpy="0 0 0" />
       <geometry>
-        <mesh filename="package://amr_fe01/meshes/chassis_l2.stl" scale="0.001 0.001 0.001" />
+        <mesh filename="package://supermarketbot/meshes/chassis_l2.stl" scale="0.001 0.001 0.001" />
       </geometry>
       <material name="base_link_material">
@@ -38,5 +38,5 @@
       <origin xyz="0 0 0" rpy="0 0 0" />
       <geometry>
-        <mesh filename="package://amr_fe01/meshes/chassis_l3.stl" scale="0.001 0.001 0.001" />
+        <mesh filename="package://supermarketbot/meshes/chassis_l3.stl" scale="0.001 0.001 0.001" />
       </geometry>
       <material name="2">
@@ -67,5 +67,5 @@
       <origin xyz="0 0 0" rpy="0 0 3.141592653589793" />
       <geometry>
-        <mesh filename="package://amr_fe01/meshes/wheel.stl" scale="0.001 0.001 0.001" />
+        <mesh filename="package://supermarketbot/meshes/wheel.stl" scale="0.001 0.001 0.001" />
       </geometry>
       <material name="3">
@@ -89,5 +89,5 @@
       <origin xyz="0 0 0" rpy="0 0 0" />
       <geometry>
-        <mesh filename="package://amr_fe01/meshes/wheel.stl" scale="0.001 0.001 0.001" />
+        <mesh filename="package://supermarketbot/meshes/wheel.stl" scale="0.001 0.001 0.001" />
       </geometry>
       <material name="4">
@@ -111,5 +111,5 @@
       <origin xyz="-0 -9e-06 -0.000115" rpy="0 0 0" />
       <geometry>
-        <mesh filename="package://amr_fe01/meshes/lidar_base_link.stl" scale="0.001 0.001 0.001" />
+        <mesh filename="package://supermarketbot/meshes/lidar_base_link.stl" scale="0.001 0.001 0.001" />
       </geometry>
       <material name="5">
@@ -201,7 +201,7 @@
       <min_angular_velocity>-1</min_angular_velocity>
       <!-- input -->
-      <topic>/amr_fe01/cmd_vel</topic>
+      <topic>/supermarketbot/cmd_vel</topic>
       <!-- output -->
-      <odom_topic>/amr_fe01/odom</odom_topic>
+      <odom_topic>/supermarketbot/odom</odom_topic>
       <tf_topic>/tf</tf_topic>
       <frame_id>odom</frame_id>
