Commit message: added the new simulator MuJoCo to simulate the robot.

File: supermarketbot/urdf/supermarketbot.urdf (robot description, URDF)
Before this commit: robot supermarketbot, 6 links, 5 joints
Links:
- link chassis_link: geometry collision box size=0.16065 0.18 0.1; collision cylinder length=0.02 radius=0.009
- link left_wheel_link: geometry collision cylinder length=0.02 radius=0.035; visual mesh filename=../meshes/wheel.stl scale=0.001 0.001 0.001
- link lidar_link: geometry collision box size=0.06 0.06 0.06; visual cylinder length=0.015 radius=0.02
- link right_wheel_link: geometry collision cylinder length=0.02 radius=0.035; visual mesh filename=../meshes/wheel.stl scale=0.001 0.001 0.001
Joints:
- joint left_wheel_link_to_chassis_link_joint: origin xyz=0.051 0.1025 0.034 rpy=0 0 0 -> xyz=0.051 0.1125 0.034 rpy=0 0 0
- joint right_wheel_link_to_chassis_link_joint: origin xyz=0.051 -0.1025 0.034 rpy=0 0 0 -> xyz=0.051 -0.0925 0.034 rpy=0 0 0
